File: FirstPCB.kicad_pcb (KiCad board)
At the start: 2 copper layers, 24 parts, among them SW1 SW_Push, U1 ATmega32U4-AU, Y1 16MHz

Commit message: Updates
Parts:
- C1, C2, C3, C4, C5, C6, C7, D1, D2, D3, D4, F1, R1, R2, R3, R4, SW1, U1, USB1, Y1: moved to B.Cu
- moved C7 106.1 mm to (91.4, 134.9)
- moved R2 99.1 mm to (77.0, 118.3), turned to 90 degrees
- moved C3 96.0 mm to (86.5, 123.8), turned to 270 degrees
- moved SW1 89.9 mm to (75.4, 140.5), turned to 180 degrees
- moved USB1 89.0 mm to (76.2, 108.7), turned to 270 degrees
- moved C6 85.2 mm to (100.0, 134.9), turned to 180 degrees
- moved R3 81.3 mm to (74.6, 118.3), turned to 90 degrees
- moved D4 75.8 mm to (145.0, 135.6), turned to 90 degrees
- moved F1 75.7 mm to (72.2, 123.6), turned to 90 degrees
- moved U1 75.0 mm to (95.7, 126.2)
- moved R1 74.8 mm to (83.3, 118.9), turned to 270 degrees
- moved C2 72.2 mm to (92.5, 115.3), turned to 90 degrees
- moved C5 66.3 mm to (87.3, 118.3), turned to 90 degrees
- moved MX1 58.8 mm to (118.2, 116.5)
- moved MX2 58.8 mm to (137.2, 116.5)
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Routing:
- net GND: track 0.00 -> 127.7 mm
- net +5V: track 0.00 -> 41.7 mm
- net Net-(R1-Pad2): track 0.00 -> 32.2 mm, vias 0 -> 2
- net Net-(R3-Pad1): track 0.00 -> 21.5 mm
- net Net-(R2-Pad1): track 0.00 -> 20.4 mm
- net ROW0: track 0.00 -> 17.6 mm
- net Net-(C2-Pad2): track 0.00 -> 10.3 mm
- net VCC: track 0.00 -> 9.97 mm
- net Net-(C1-Pad2): track 0.00 -> 8.27 mm
- net Net-(D2-Pad2): track 0.00 -> 6.52 mm
- net Net-(C3-Pad1): track 0.00 -> 5.23 mm
- net D-: track 0.00 -> 4.45 mm
- net D+: track 0.00 -> 4.44 mm
- net Net-(R4-Pad1): track 0.00 -> 3.73 mm
Other:
- board outline added: 77.6 x 38.2 mm
- net class Default: trace_width 0.25 -> 0.254
- net class Power added: clearance 0.2, trace_width 0.381, via_dia 0.8, via_drill 0.4
