File: FirstPCB.sch (KiCad schematic (older format))
At the start: 24 parts, among them SW1 SW_Push, U1 ATmega32U4-AU, Y1 16MHz

Commit message: Updates
Parts:
- D1, D2, D3, D4: footprint Diode_SMD:D_SOD-123 -> (none)
- MX1, MX2, MX3, MX4: footprint MX_Alps_Hybrid:MX-1U-NoLED -> (none)
Connections:
- net COL0: now also U1.29 (PB5); no longer U1.28 (PB4)
- net COL1: now also U1.28 (PB4); no longer U1.29 (PB5)
Changed lines of the file:
@@
 	2500 3400 2800 3400
-$Comp
-L power:+5V #PWR0111
-U 1 1 60B0A1A4
-P 1850 2800
-F 0 "#PWR0111" H 1850 2650 50  0001 C CNN
-F 1 "+5V" H 1865 2973 50  0000 C CNN
-F 2 "" H 1850 2800 50  0001 C CNN
-F 3 "" H 1850 2800 50  0001 C CNN
-	1    1850 2800
-	1    0    0    -1
-$EndComp
-$Comp
-L power:GND #PWR0112
-U 1 1 60B0B473
-P 2100 2700
-F 0 "#PWR0112" H 2100 2450 50  0001 C CNN
-F 1 "GND" H 2105 2527 50  0000 C CNN
-F 2 "" H 2100 2700 50  0001 C CNN
-F 3 "" H 2100 2700 50  0001 C CNN
-	1    2100 2700
-	1    0    0    -1
-$EndComp
 $Comp
 L power:+5V #PWR0113
@@
 Wire Wire Line
 	2650 3800 2650 3950
-$Comp
-L Device:D_Small D1
-U 1 1 60B1ADA0
-P 8000 2950
-F 0 "D1" V 8046 2880 50  0000 R CNN
-F 1 "D_Small" V 7955 2880 50  0000 R CNN
-F 2 "Diode_SMD:D_SOD-123" V 8000 2950 50  0001 C CNN
-F 3 "~" V 8000 2950 50  0001 C CNN
-	1    8000 2950
-	0    -1   -1   0
-$EndComp
-$Comp
-L MX_Alps_Hybrid:MX-NoLED MX1
-U 1 1 60B24CBD
-P 8150 2700
-F 0 "MX1" H 8183 2923 60  0000 C CNN
-F 1 "MX-NoLED" H 8183 2849 20  0000 C CNN
-F 2 "MX_Alps_Hybrid:MX-1U-NoLED" H 7525 2675 60  0001 C CNN
-F 3 "" H 7525 2675 60  0001 C CNN
-	1    8150 2700
-	1    0    0    -1
-$EndComp
 Wire Wire Line
-	8100 2850 8000 2850
-$Comp
-L Device:D_Small D2
-U 1 1 60B26BEF
-P 8450 2950
-F 0 "D2" V 8496 2880 50  0000 R CNN
-F 1 "D_Small" V 8405 2880 50  0000 R CNN
-F 2 "Diode_SMD:D_SOD-123" V 8450 2950 50  0001 C CNN
-F 3 "~" V 8450 2950 50  0001 C CNN
-	1    8450 2950
-	0    -1   -1   0
-$EndComp
-$Comp
-L MX_Alps_Hybrid:MX-NoLED MX2
-U 1 1 60B26BF9
-P 8600 2700
-F 0 "MX2" H 8633 2923 60  0000 C CNN
-F 1 "MX-NoLED" H 8633 2849 20  0000 C CNN
-F 2 "MX_Alps_Hybrid:MX-1U-NoLED" H 7975 2675 60  0001 C CNN
-F 3 "" H 7975 2675 60  0001 C CNN
-	1    8600 2700
-	1    0    0    -1
-$EndComp
+	7550 3150 7900 3150
 Wire Wire Line
-	8550 2850 8450 2850
-$Comp
-L Device:D_Small D3
-U 1 1 60B292F1
-P 8000 3600
-F 0 "D3" V 8046 3530 50  0000 R CNN
-F 1 "D_Small" V 7955 3530 50  0000 R CNN
-F 2 "Diode_SMD:D_SOD-123" V 8000 3600 50  0001 C CNN
-F 3 "~" V 8000 3600 50  0001 C CNN
-	1    8000 3600
-	0    -1   -1   0
-$EndComp
-$Comp
-L MX_Alps_Hybrid:MX-NoLED MX3
-U 1 1 60B292FB
-P 8150 3350
-F 0 "MX3" H 8183 3573 60  0000 C CNN
-F 1 "MX-NoLED" H 8183 3499 20  0000 C CNN
-F 2 "MX_Alps_Hybrid:MX-1U-NoLED" H 7525 3325 60  0001 C CNN
-F 3 "" H 7525 3325 60  0001 C CNN
-	1    8150 3350
-	1    0    0    -1
-$EndComp
-Wire Wire Line
-	8100 3500 8000 3500
-$Comp
-L Device:D_Small D4
-U 1 1 60B29306
-P 8450 3600
-F 0 "D4" V 8496 3530 50  0000 R CNN
-F 1 "D_Small" V 8405 3530 50  0000 R CNN
-F 2 "Diode_SMD:D_SOD-123" V 8450 3600 50  0001 C CNN
-F 3 "~" V 8450 3600 50  0001 C CNN
-	1    8450 3600
-	0    -1   -1   0
-$EndComp
-$Comp
-L MX_Alps_Hybrid:MX-NoLED MX4
-U 1 1 60B29310
-P 8600 3350
-F 0 "MX4" H 8633 3573 60  0000 C CNN
-F 1 "MX-NoLED" H 8633 3499 20  0000 C CNN
-F 2 "MX_Alps_Hybrid:MX-1U-NoLED" H 7975 3325 60  0001 C CNN
-F 3 "" H 7975 3325 60  0001 C CNN
-	1    8600 3350
-	1    0    0    -1
-$EndComp
-Wire Wire Line
-	8550 3500 8450 3500
-Wire Wire Line
-	8300 2400 8300 2650
-Connection ~ 8300 2650
-Wire Wire Line
-	8750 2400 8750 2650
-Connection ~ 8750 2650
-Wire Wire Line
-	8750 2650 8750 3300
-Wire Wire Line
-	8300 2650 8300 3300
-Wire Wire Line
-	7650 3050 8000 3050
-Connection ~ 8000 3050
-Wire Wire Line
-	8000 3050 8450 3050
-Wire Wire Line
-	8450 3700 8000 3700
-Connection ~ 8000 3700
-Wire Wire Line
-	8000 3700 7650 3700
-Text GLabel 8300 2400 1    50   Input ~ 0
+	7900 3800 7550 3800
+Text GLabel 8200 2500 1    50   Input ~ 0
 COL0
-Text GLabel 8750 2400 1    50   Input ~ 0
-COL1
-Text GLabel 7650 3050 0    50   Input ~ 0
+Text GLabel 7550 3150 0    50   Input ~ 0
 ROW0
-Text GLabel 7650 3700 0    50   Input ~ 0
+Text GLabel 7550 3800 0    50   Input ~ 0
 ROW1
 Text GLabel 6500 4400 2    50   Input ~ 0
@@
 Text GLabel 6500 3100 2    50   Input ~ 0
 ROW1
+Text GLabel 6500 3000 2    50   Input ~ 0
+COL0
 Text GLabel 6500 2900 2    50   Input ~ 0
-COL0
-Text GLabel 6500 3000 2    50   Input ~ 0
 COL1
+Text GLabel 8800 2500 1    50   Input ~ 0
+COL1
+$Comp
+L MX_Alps_Hybrid:MX-NoLED MX3
+U 1 1 60C03038
+P 8050 3450
+F 0 "MX3" H 8083 3673 60  0000 C CNN
+F 1 "MX-NoLED" H 8083 3599 20  0000 C CNN
+F 2 "" H 7425 3425 60  0001 C CNN
+F 3 "" H 7425 3425 60  0001 C CNN
+	1    8050 3450
+	1    0    0    -1
+$EndComp
+$Comp
+L Device:D_Small D3
+U 1 1 60C252F1
+P 7900 3700
+F 0 "D3" V 7946 3630 50  0000 R CNN
+F 1 "D_Small" V 7855 3630 50  0000 R CNN
+F 2 "" V 7900 3700 50  0001 C CNN
+F 3 "~" V 7900 3700 50  0001 C CNN
+	1    7900 3700
+	0    -1   -1   0
+$EndComp
+$Comp
+L MX_Alps_Hybrid:MX-NoLED MX4
+U 1 1 60C278F6
+P 8650 3450
+F 0 "MX4" H 8683 3673 60  0000 C CNN
+F 1 "MX-NoLED" H 8683 3599 20  0000 C CNN
+F 2 "" H 8025 3425 60  0001 C CNN
+F 3 "" H 8025 3425 60  0001 C CNN
+	1    8650 3450
+	1    0    0    -1
+$EndComp
+$Comp
+L MX_Alps_Hybrid:MX-NoLED MX1
+U 1 1 60C28069
+P 8050 2800
+F 0 "MX1" H 8083 3023 60  0000 C CNN
+F 1 "MX-NoLED" H 8083 2949 20  0000 C CNN
+F 2 "" H 7425 2775 60  0001 C CNN
+F 3 "" H 7425 2775 60  0001 C CNN
+	1    8050 2800
+	1    0    0    -1
+$EndComp
+$Comp
+L MX_Alps_Hybrid:MX-NoLED MX2
+U 1 1 60C282F4
+P 8650 2800
+F 0 "MX2" H 8683 3023 60  0000 C CNN
+F 1 "MX-NoLED" H 8683 2949 20  0000 C CNN
+F 2 "" H 8025 2775 60  0001 C CNN
+F 3 "" H 8025 2775 60  0001 C CNN
+	1    8650 2800
+	1    0    0    -1
+$EndComp
+$Comp
+L Device:D_Small D4
+U 1 1 60C28657
+P 8500 3700
+F 0 "D4" V 8546 3630 50  0000 R CNN
+F 1 "D_Small" V 8455 3630 50  0000 R CNN
+F 2 "" V 8500 3700 50  0001 C CNN
+F 3 "~" V 8500 3700 50  0001 C CNN
+	1    8500 3700
+	0    -1   -1   0
+$EndComp
+$Comp
+L Device:D_Small D1
+U 1 1 60C288C0
+P 7900 3050
+F 0 "D1" V 7946 2980 50  0000 R CNN
+F 1 "D_Small" V 7855 2980 50  0000 R CNN
+F 2 "" V 7900 3050 50  0001 C CNN
+F 3 "~" V 7900 3050 50  0001 C CNN
+	1    7900 3050
+	0    -1   -1   0
+$EndComp
+$Comp
+L Device:D_Small D2
+U 1 1 60C28AFC
+P 8500 3050
+F 0 "D2" V 8546 2980 50  0000 R CNN
+F 1 "D_Small" V 8455 2980 50  0000 R CNN
+F 2 "" V 8500 3050 50  0001 C CNN
+F 3 "~" V 8500 3050 50  0001 C CNN
+	1    8500 3050
+	0    -1   -1   0
+$EndComp
+Wire Wire Line
+	8200 2500 8200 2750
+Connection ~ 8200 2750
+Wire Wire Line
+	8200 2750 8200 3400
+Wire Wire Line
+	8500 3800 7900 3800
+Connection ~ 7900 3800
+Wire Wire Line
+	8800 2500 8800 2750
+Connection ~ 8800 2750
+Wire Wire Line
+	8800 2750 8800 3400
+Wire Wire Line
+	8000 2950 7900 2950
+Wire Wire Line
+	8600 2950 8500 2950
+Wire Wire Line
+	8600 3600 8500 3600
+Wire Wire Line
+	8000 3600 7900 3600
+Wire Wire Line
+	8500 3150 7900 3150
+Connection ~ 7900 3150
 $EndSCHEMATC

Commit message: Converted to USB Type-C
Parts:
- removed R2, R3: 22, Resistor_SMD:R_0805_2012Metric, symbol Device:R_Small
- removed USB1: Molex-0548190589, random-keyboard-parts:Molex-0548190589, symbol random-keyboard-parts:Molex-0548190589
- added R5, R6: 22, Resistor_SMD:R_0805_2012Metric, symbol Device:R_Small
- added R7, R8: 5.1k, Resistor_SMD:R_0805_2012Metric, symbol Device:R_Small
- added U2: PRTR5V0U2X, locallib:SOT143B, symbol random-keyboard-parts:PRTR5V0U2X
- added USB1: HRO-TYPE-C-31-M-12, Type-C:HRO-TYPE-C-31-M-12-Assembly, symbol Type-C:HRO-TYPE-C-31-M-12
- D1, D2, D3, D4: footprint (none) -> Diode_SMD:D_SOD-123
- MX1, MX2, MX3, MX4: footprint (none) -> MX_Only:MXOnly-1U-NoLED
Connections:
- net D+: now also U1.4 (D+), R6.1
- net D-: now also U1.3 (D-), R5.1
- net GND: now also R7.1, R8.1, U2.1 (GND), USB1.1 (GND), USB1.12 (GND), USB1.13 (SHIELD)
- net VCC: now also U2.4 (VCC), USB1.11 (VBUS), USB1.2 (VBUS)
- new net: R8.2, USB1.10 (CC2)
- new net: R7.2, USB1.4 (CC1)
- new net: R5.2, U2.3 (IO2), USB1.5 (DN2), USB1.7 (DN1)
- new net: R6.2, U2.2 (IO1), USB1.6 (DP1), USB1.8 (DP2)
